File: 4_7_SEGMENT.sch (KiCad schematic (older format))
At the start: 19 parts

Commit message: Add files via upload
Parts:
- AFF1: renamed from AFF?; footprint (none) -> Displays_7-Segment:Cx56-12
- P12: renamed from P?; footprint (none) -> Pin_Headers:Pin_Header_Straight_1x04
- P13: renamed from P?; footprint (none) -> Pin_Headers:Pin_Header_Straight_1x08
- Q1, Q2, Q3, Q4: renamed from Q?; footprint TO-92 -> TO_SOT_Packages_THT:TO-92_Inline_Wide
- R11, R12, R13, R14, R15, R16, R17, R18, R19, R20, R21, R22: renamed from R?; footprint (none) -> Resistors_ThroughHole:Resistor_Horizontal_RM10mm
Changed lines of the file:
@@
 EESchema Schematic File Version 2
+LIBS:8051_dev-rescue
 LIBS:power
 LIBS:device
@@
 LIBS:contrib
 LIBS:valves
-LIBS:8051_generic_89s51
 LIBS:7805_mod
-LIBS:HexConverter
-LIBS:MOTOR
-LIBS:ams1117_
-LIBS:arduinoNano
-LIBS:arduinouno
-LIBS:buzzer
-LIBS:cmos_cell
-LIBS:color_sensor
-LIBS:esp8266
-LIBS:fingerprintsensor
-LIBS:flex
-LIBS:ftdi232rl
-LIBS:hexconverter
-LIBS:i2cmemoty24ls256
-LIBS:l293d_modified
-LIBS:ldr
-LIBS:lm3915
-LIBS:oleddisplay
-LIBS:ov7670
-LIBS:pushbutton
-LIBS:relay
-LIBS:sd_card_module
-LIBS:servo
-LIBS:valve
-LIBS:xbee
-LIBS:max_232
-LIBS:0808
 LIBS:8051_dev-cache
 EELAYER 25 0
@@
 $Descr A4 11693 8268
 encoding utf-8
-Sheet 6 9
+Sheet 6 10
 Title ""
 Date ""
@@
 $EndDescr
 $Comp
-L BC547 Q?
+L BC547 Q1
 U 1 1 579B4E8D
 P 4650 3050
-F 0 "Q?" H 4450 2750 50  0000 L CNN
+F 0 "Q1" H 4450 2750 50  0000 L CNN
 F 1 "BC547" H 4450 2850 50  0000 L CNN
-F 2 "TO-92" H 4450 2800 50  0000 L CIN
+F 2 "TO_SOT_Packages_THT:TO-92_Inline_Wide" H 4450 2800 50  0000 L CIN
 F 3 "" H 4650 3050 50  0000 L CNN
 	1    4650 3050
@@
 $EndComp
 $Comp
-L R R?
+L R R11
 U 1 1 579B4ECC
 P 4450 2750
-F 0 "R?" V 4530 2750 50  0000 C CNN
+F 0 "R11" V 4530 2750 50  0000 C CNN
 F 1 "50K" V 4450 2750 50  0000 C CNN
-F 2 "" V 4380 2750 50  0000 C CNN
+F 2 "Resistors_ThroughHole:Resistor_Horizontal_RM10mm" V 4380 2750 50  0001 C CNN
 F 3 "" H 4450 2750 50  0000 C CNN
 	1    4450 2750
@@
 $EndComp
 $Comp
-L BC547 Q?
+L BC547 Q2
 U 1 1 579B4FF0
 P 5150 3050
-F 0 "Q?" H 4950 2750 50  0000 L CNN
+F 0 "Q2" H 4950 2750 50  0000 L CNN
 F 1 "BC547" H 4950 2850 50  0000 L CNN
-F 2 "TO-92" H 4950 2800 50  0000 L CIN
+F 2 "TO_SOT_Packages_THT:TO-92_Inline_Wide" H 4950 2800 50  0000 L CIN
 F 3 "" H 5150 3050 50  0000 L CNN
 	1    5150 3050
@@
 $EndComp
 $Comp
-L BC547 Q?
+L BC547 Q3
 U 1 1 579B5022
 P 5650 3050
-F 0 "Q?" H 5500 2700 50  0000 L CNN
+F 0 "Q3" H 5500 2700 50  0000 L CNN
 F 1 "BC547" H 5450 2900 50  0000 L CNN
-F 2 "TO-92" H 5450 2800 50  0000 L CIN
+F 2 "TO_SOT_Packages_THT:TO-92_Inline_Wide" H 5450 2800 50  0000 L CIN
 F 3 "" H 5650 3050 50  0000 L CNN
 	1    5650 3050
@@
 $EndComp
 $Comp
-L BC547 Q?
+L BC547 Q4
 U 1 1 579B505F
 P 6150 3050
-F 0 "Q?" H 5950 2750 50  0000 L CNN
+F 0 "Q4" H 5950 2750 50  0000 L CNN
 F 1 "BC547" H 5900 2900 50  0000 L CNN
-F 2 "TO-92" H 5950 2850 50  0000 L CIN
+F 2 "TO_SOT_Packages_THT:TO-92_Inline_Wide" H 5950 2850 50  0000 L CIN
 F 3 "" H 6150 3050 50  0000 L CNN
 	1    6150 3050
@@
 	6250 3250 6250 3400
 $Comp
-L R R?
+L R R12
 U 1 1 579B54A6
 P 4950 2750
-F 0 "R?" V 5030 2750 50  0000 C CNN
+F 0 "R12" V 5030 2750 50  0000 C CNN
 F 1 "50K" V 4950 2750 50  0000 C CNN
-F 2 "" V 4880 2750 50  0000 C CNN
+F 2 "Resistors_ThroughHole:Resistor_Horizontal_RM10mm" V 4880 2750 50  0001 C CNN
 F 3 "" H 4950 2750 50  0000 C CNN
 	1    4950 2750
@@
 $EndComp
 $Comp
-L R R?
+L R R16
 U 1 1 579B54DD
 P 5450 2750
-F 0 "R?" V 5530 2750 50  0000 C CNN
+F 0 "R16" V 5530 2750 50  0000 C CNN
 F 1 "50K" V 5450 2750 50  0000 C CNN
-F 2 "" V 5380 2750 50  0000 C CNN
+F 2 "Resistors_ThroughHole:Resistor_Horizontal_RM10mm" V 5380 2750 50  0001 C CNN
 F 3 "" H 5450 2750 50  0000 C CNN
 	1    5450 2750
@@
 $EndComp
 $Comp
-L R R?
+L R R22
 U 1 1 579B5515
 P 5950 2750
-F 0 "R?" V 6030 2750 50  0000 C CNN
+F 0 "R22" V 6030 2750 50  0000 C CNN
 F 1 "50K" V 5950 2750 50  0000 C CNN
-F 2 "" V 5880 2750 50  0000 C CNN
+F 2 "Resistors_ThroughHole:Resistor_Horizontal_RM10mm" V 5880 2750 50  0001 C CNN
 F 3 "" H 5950 2750 50  0000 C CNN
 	1    5950 2750
@@
 Connection ~ 6250 2300
 $Comp
-L CONN_01X04 P?
+L CONN_01X04 P12
 U 1 1 579B5726
 P 5250 1800
-F 0 "P?" H 5250 2050 50  0000 C CNN
+F 0 "P12" H 5250 2050 50  0000 C CNN
 F 1 "4_7_SEGMENT_BC547_CONTROL" V 5350 1800 50  0000 C CNN
-F 2 "" H 5250 1800 50  0000 C CNN
+F 2 "Pin_Headers:Pin_Header_Straight_1x04" H 5250 1800 50  0001 C CNN
 F 3 "" H 5250 1800 50  0000 C CNN
 	1    5250 1800
@@
 	5950 2000 5950 2600
 $Comp
-L CONN_01X08 P?
+L CONN_01X08 P13
 U 1 1 579B5961
 P 5500 6000
-F 0 "P?" H 5500 6450 50  0000 C CNN
+F 0 "P13" H 5500 6450 50  0000 C CNN
 F 1 "4_7_SEGMENT_HEADER" V 5600 6000 50  0000 C CNN
-F 2 "" H 5500 6000 50  0000 C CNN
+F 2 "Pin_Headers:Pin_Header_Straight_1x08" H 5500 6000 50  0001 C CNN
 F 3 "" H 5500 6000 50  0000 C CNN
 	1    5500 6000
@@
 	5850 5800 5850 5100
 $Comp
-L R R?
+L R R13
 U 1 1 579B6021
 P 5150 4950
-F 0 "R?" V 5230 4950 50  0000 C CNN
+F 0 "R13" V 5230 4950 50  0000 C CNN
 F 1 "330" V 5150 4950 50  0000 C CNN
-F 2 "" V 5080 4950 50  0000 C CNN
+F 2 "Resistors_ThroughHole:Resistor_Horizontal_RM10mm" V 5080 4950 50  0001 C CNN
 F 3 "" H 5150 4950 50  0000 C CNN
 	1    5150 4950
@@
 $EndComp
 $Comp
-L R R?
+L R R14
 U 1 1 579B612E
 P 5250 4950
-F 0 "R?" V 5330 4950 50  0000 C CNN
+F 0 "R14" V 5330 4950 50  0000 C CNN
 F 1 "330" V 5250 4950 50  0000 C CNN
-F 2 "" V 5180 4950 50  0000 C CNN
+F 2 "Resistors_ThroughHole:Resistor_Horizontal_RM10mm" V 5180 4950 50  0001 C CNN
 F 3 "" H 5250 4950 50  0000 C CNN
 	1    5250 4950
@@
 $EndComp
 $Comp
-L R R?
+L R R15
 U 1 1 579B6169
 P 5350 4950
-F 0 "R?" V 5430 4950 50  0000 C CNN
+F 0 "R15" V 5430 4950 50  0000 C CNN
 F 1 "330" V 5350 4950 50  0000 C CNN
-F 2 "" V 5280 4950 50  0000 C CNN
+F 2 "Resistors_ThroughHole:Resistor_Horizontal_RM10mm" V 5280 4950 50  0001 C CNN
 F 3 "" H 5350 4950 50  0000 C CNN
 	1    5350 4950
@@
 $EndComp
 $Comp
-L R R?
+L R R17
 U 1 1 579B61FD
 P 5450 4950
-F 0 "R?" V 5530 4950 50  0000 C CNN
+F 0 "R17" V 5530 4950 50  0000 C CNN
 F 1 "330" V 5450 4950 50  0000 C CNN
-F 2 "" V 5380 4950 50  0000 C CNN
+F 2 "Resistors_ThroughHole:Resistor_Horizontal_RM10mm" V 5380 4950 50  0001 C CNN
 F 3 "" H 5450 4950 50  0000 C CNN
 	1    5450 4950
@@
 $EndComp
 $Comp
-L R R?
+L R R18
 U 1 1 579B6203
 P 5550 4950
-F 0 "R?" V 5630 4950 50  0000 C CNN
+F 0 "R18" V 5630 4950 50  0000 C CNN
 F 1 "330" V 5550 4950 50  0000 C CNN
-F 2 "" V 5480 4950 50  0000 C CNN
+F 2 "Resistors_ThroughHole:Resistor_Horizontal_RM10mm" V 5480 4950 50  0001 C CNN
 F 3 "" H 5550 4950 50  0000 C CNN
 	1    5550 4950
@@
 $EndComp
 $Comp
-L R R?
+L R R19
 U 1 1 579B6209
 P 5650 4950
-F 0 "R?" V 5730 4950 50  0000 C CNN
+F 0 "R19" V 5730 4950 50  0000 C CNN
 F 1 "330" V 5650 4950 50  0000 C CNN
-F 2 "" V 5580 4950 50  0000 C CNN
+F 2 "Resistors_ThroughHole:Resistor_Horizontal_RM10mm" V 5580 4950 50  0001 C CNN
 F 3 "" H 5650 4950 50  0000 C CNN
 	1    5650 4950
@@
 $EndComp
 $Comp
-L R R?
+L R R20
 U 1 1 579B628D
 P 5750 4950
-F 0 "R?" V 5830 4950 50  0000 C CNN
+F 0 "R20" V 5830 4950 50  0000 C CNN
 F 1 "330" V 5750 4950 50  0000 C CNN
-F 2 "" V 5680 4950 50  0000 C CNN
+F 2 "Resistors_ThroughHole:Resistor_Horizontal_RM10mm" V 5680 4950 50  0001 C CNN
 F 3 "" H 5750 4950 50  0000 C CNN
 	1    5750 4950
@@
 $EndComp
 $Comp
-L R R?
+L R R21
 U 1 1 579B6293
 P 5850 4950
-F 0 "R?" V 5930 4950 50  0000 C CNN
+F 0 "R21" V 5930 4950 50  0000 C CNN
 F 1 "330" V 5850 4950 50  0000 C CNN
-F 2 "" V 5780 4950 50  0000 C CNN
+F 2 "Resistors_ThroughHole:Resistor_Horizontal_RM10mm" V 5780 4950 50  0001 C CNN
 F 3 "" H 5850 4950 50  0000 C CNN
 	1    5850 4950
@@
 $EndComp
 $Comp
-L CC56-12 AFF?
+L CC56-12 AFF1
 U 1 1 579B76F1
 P 5450 4100
-F 0 "AFF?" H 5450 4550 50  0000 C CNN
+F 0 "AFF1" H 5450 4550 50  0000 C CNN
 F 1 "CC56-12" H 5450 4350 50  0000 C CNN
-F 2 "" H 4950 4100 50  0000 C CNN
+F 2 "Displays_7-Segment:Cx56-12" H 4950 4100 50  0001 C CNN
 F 3 "" H 4950 4100 50  0000 C CNN
 	1    5450 4100
