File: 8051_dev.sch (KiCad schematic (older format))
At the start: 12 parts

Commit message: Add files via upload
Parts:
- removed U?: 8051_generic_89s51, symbol 8051_generic_89s51
- added U1: 8051_generic_89s51, Housings_DIP:DIP-40_W15.24mm_LongPads, symbol 8051_generic_89s51
- C1, C2, C3: renamed from C?; footprint (none) -> Capacitors_ThroughHole:C_Disc_D3_P2.5
- P1, P2, P3, P4: renamed from P?; footprint (none) -> Pin_Headers:Pin_Header_Straight_1x08
- R1: renamed from R?; footprint (none) -> Resistors_ThroughHole:Resistor_Horizontal_RM10mm
- RR1: renamed from RR?; footprint (none) -> Resistors_ThroughHole:Resistor_Array_SIP8
- SW1: renamed from SW?; footprint (none) -> Buttons_Switches_ThroughHole:Push_button_2_pin
- Y1: renamed from Y?; footprint (none) -> Crystals:HC-49V
Connections:
- net GND: now also C1.2, C2.2, U1.20 (GND)
- net VCC: now also U1.31 (EA/VPP), U1.40 (VCC)
- net x1: now also U1.19 (XTAL1)
- net x2: now also U1.18 (XTAL2)
- net at P2.8 (P8): now also U1.1 (P1.0)
- net at P1.8 (P8): now also U1.10 (P3.0_RX)
- net at P1.7 (P7): now also U1.11 (P3.0_TX)
- net at P1.6 (P6): now also U1.12 (INT0)
- net at P1.5 (P5): now also U1.13 (INT1)
- net at P1.4 (P4): now also U1.14 (T0)
- net at P1.3 (P3): now also U1.15 (T1)
- net at P1.2 (P2): now also U1.16 (WR)
- net at P1.1 (P1): now also U1.17 (RD)
- net at P2.7 (P7): now also U1.2 (P1.1)
- net at P3.8 (P8): now also U1.21 (A8)
- net at P3.7 (P7): now also U1.22 (A9)
- net at P3.6 (P6): now also U1.23 (A10)
- net at P3.5 (P5): now also U1.24 (A11)
- net at P3.4 (P4): now also U1.25 (A12)
- net at P3.3 (P3): now also U1.26 (A13)
- net at P3.2 (P2): now also U1.27 (A14)
- net at P3.1 (P1): now also U1.28 (A15)
- net at P2.6 (P6): now also U1.3 (P1.2)
- net at P4.8 (P8), RR1.9: now also U1.32 (AD7)
- net at P4.7 (P7), RR1.8: now also U1.33 (AD6)
- net at P4.6 (P6), RR1.7: now also U1.34 (AD5)
- net at P4.5 (P5), RR1.6: now also U1.35 (AD4)
- net at P4.4 (P4), RR1.5: now also U1.36 (AD3)
- net at P4.3 (P3), RR1.4: now also U1.37 (AD2)
- net at P4.2 (P2), RR1.3: now also U1.38 (AD1)
- net at P4.1 (P1), RR1.2: now also U1.39 (AD0)
- net at P2.5 (P5): now also U1.4 (P1.3)
- net at P2.4 (P4): now also U1.5 (P1.4)
- net at P2.3 (P3): now also U1.6 (P1.5_mosi)
- net at P2.2 (P2): now also U1.7 (P1.6_miso)
- net at P2.1 (P1): now also U1.8 (P1.7_sck)
- net at C3.2, R1.1, SW1.1: now also U1.9 (RST)
Other:
- moved on the sheet: P4, RR1
