File: ADC.sch (KiCad schematic (older format))
At the start: 5 parts

Commit message: Add files via upload
Parts:
- removed P?: ADC_CONTROLE, symbol CONN_01X08
- removed P?: ADC_IN_ANALOG, symbol CONN_01X08
- removed U?: 0808, symbol 0808
- added P17: ADC_power_head, Pin_Headers:Pin_Header_Straight_1x02, symbol CONN_01X02
- added P18: ADCC1, Pin_Headers:Pin_Header_Straight_1x04, symbol CONN_01X04
- added P19: ADCV_1, Pin_Headers:Pin_Header_Straight_1x03, symbol CONN_01X03
- added P28: ADCV_2, Pin_Headers:Pin_Header_Straight_1x05, symbol CONN_01X05
- added P29: ADCC2, Pin_Headers:Pin_Header_Straight_1x04, symbol CONN_01X04
- added U4: 0808, Housings_DIP:DIP-28_W15.24mm_LongPads, symbol 0808
- P20: renamed from P?; footprint (none) -> Pin_Headers:Pin_Header_Straight_1x08
- RV2: renamed from RV?; footprint (none) -> Potentiometers:Potentiometer_Trimmer-Suntan-TSR-3386P
Connections:
- net ADC_GND: now also P17.1 (P1), U4.13 (GND), U4.16 (VREF-)
- net ADC_VCC: now also P17.2 (P2), U4.11 (VCC), U4.12 (vREF+)
- net IN0: now also P19.3 (P3), U4.26 (IN0)
- net IN1: now also P19.2 (P2), U4.27 (IN1)
- net IN2: now also P19.1 (P1), U4.28 (IN2)
- net IN3: now also P28.5 (P5), U4.1 (IN3)
- net IN4: now also P28.4 (P4), U4.2 (IN4)
- net IN5: now also P28.3 (P3), U4.3 (IN5)
- net IN6: now also P28.2 (P2), U4.4 (IN6)
- net IN7: now also P28.1 (P1), U4.5 (IN7)
- net at P20.7 (P7): now also U4.14 (2-7)
- net at P20.6 (P6): now also U4.15 (2-6)
- net at P20.8 (P8): now also U4.17 (2-8)
- net at P20.4 (P4): now also U4.18 (2-4)
- net at P20.3 (P3): now also U4.19 (2-3)
- net at P20.2 (P2): now also U4.20 (2-2)
- net at P20.1 (P1): now also U4.21 (2-1)
- net at P20.5 (P5): now also U4.8 (2-5)
- new net: P18.1 (P1), U4.22 (ALE)
- new net: P18.2 (P2), U4.23 (ADD_C)
- new net: P18.3 (P3), U4.24 (ADD_B)
- new net: P18.4 (P4), U4.25 (ADD_A)
- new net: P29.1 (P1), U4.10 (CLOCK)
- new net: P29.4 (P4), U4.6 (START)
- new net: P29.3 (P3), U4.7 (EOC)
- new net: P29.2 (P2), U4.9 (OUTeN)
