File: DCMotor.sch (KiCad schematic (older format))
At the start: 3 parts

Commit message: Add files via upload
Parts:
- added P16: DC_motor_power_head, Pin_Headers:Pin_Header_Straight_1x02, symbol CONN_01X02
- P14: renamed from P?; footprint (none) -> Pin_Headers:Pin_Header_Straight_1x04
- P15: renamed from P?; footprint (none) -> Pin_Headers:Pin_Header_Straight_1x02
- U3: renamed from U?; footprint (none) -> Housings_DIP:DIP-16_W7.62mm_LongPads
Connections:
- net L293D_GND: now also P16.2 (P2)
- net L293D_VCC: no longer names the net of U3.1 (EnA), U3.16 (VCC), U3.9 (EnB)
- net L293D_VCC: now also P16.1 (P1)
Changed lines of the file:
@@
 EESchema Schematic File Version 2
+LIBS:8051_dev-rescue
 LIBS:power
 LIBS:device
@@
 LIBS:contrib
 LIBS:valves
-LIBS:8051_generic_89s51
 LIBS:7805_mod
-LIBS:HexConverter
-LIBS:MOTOR
-LIBS:ams1117_
-LIBS:arduinoNano
-LIBS:arduinouno
-LIBS:buzzer
-LIBS:cmos_cell
-LIBS:color_sensor
-LIBS:esp8266
-LIBS:fingerprintsensor
-LIBS:flex
-LIBS:ftdi232rl
-LIBS:hexconverter
-LIBS:i2cmemoty24ls256
-LIBS:l293d_modified
-LIBS:ldr
-LIBS:lm3915
-LIBS:oleddisplay
-LIBS:ov7670
-LIBS:pushbutton
-LIBS:relay
-LIBS:sd_card_module
-LIBS:servo
-LIBS:valve
-LIBS:xbee
-LIBS:max_232
-LIBS:0808
 LIBS:8051_dev-cache
 EELAYER 25 0
@@
 $Descr A4 11693 8268
 encoding utf-8
-Sheet 8 9
+Sheet 6 10
 Title ""
 Date ""
@@
 $EndDescr
 $Comp
-L L293D_modified U?
+L L293D_modified U3
 U 1 1 579BAE26
 P 4500 4000
-F 0 "U?" H 4500 4000 60  0000 C CNN
+F 0 "U3" H 4500 4000 60  0000 C CNN
 F 1 "L293D_modified" H 4500 5000 60  0000 C CNN
-F 2 "" H 4500 4000 60  0000 C CNN
+F 2 "Housings_DIP:DIP-16_W7.62mm_LongPads" H 4500 4000 60  0001 C CNN
 F 3 "" H 4500 4000 60  0000 C CNN
 	1    4500 4000
 	1    0    0    -1
 $EndComp
-Text HLabel 5100 2600 2    60   Input Italic 0
-L293D_VCC
-Text HLabel 6250 3500 2    60   Input Italic 0
-L239D_GND
 Text GLabel 6050 3500 0    60   Input Italic 0
 L293D_GND
@@
 L293D_GND
 Wire Wire Line
-	5100 2600 4050 2600
+	4050 2600 6350 2600
 Wire Wire Line
 	4050 2600 4050 3150
@@
 	5100 3550 4950 3550
 Wire Wire Line
-	6050 3500 6250 3500
+	6250 3500 6050 3500
 Connection ~ 3900 3550
 Wire Wire Line
@@
 	5400 2900 4950 2900
 $Comp
-L CONN_01X04 P?
+L CONN_01X04 P14
 U 1 1 579BB340
 P 2350 3500
-F 0 "P?" H 2350 3750 50  0000 C CNN
+F 0 "P14" H 2350 3750 50  0000 C CNN
 F 1 "L293D_HEADER" V 2450 3500 50  0000 C CNN
-F 2 "" H 2350 3500 50  0000 C CNN
+F 2 "Pin_Headers:Pin_Header_Straight_1x04" H 2350 3500 50  0001 C CNN
 F 3 "" H 2350 3500 50  0000 C CNN
 	1    2350 3500
@@
 	2700 3650 2550 3650
 $Comp
-L CONN_01X02 P?
+L CONN_01X02 P15
 U 1 1 579BB5E5
 P 3950 4300
-F 0 "P?" H 3950 4450 50  0000 C CNN
+F 0 "P15" H 3950 4450 50  0000 C CNN
 F 1 "L293D_9V" V 4050 4300 50  0000 C CNN
-F 2 "" H 3950 4300 50  0000 C CNN
+F 2 "Pin_Headers:Pin_Header_Straight_1x02" H 3950 4300 50  0001 C CNN
 F 3 "" H 3950 4300 50  0000 C CNN
 	1    3950 4300
@@
 Wire Wire Line
 	3900 3950 3900 4100
+$Comp
+L CONN_01X02 P16
+U 1 1 57A5E953
+P 6550 2700
+F 0 "P16" H 6550 2850 50  0000 C CNN
+F 1 "DC_motor_power_head" V 6650 2700 50  0000 C CNN
+F 2 "Pin_Headers:Pin_Header_Straight_1x02" H 6550 2700 50  0001 C CNN
+F 3 "" H 6550 2700 50  0000 C CNN
+	1    6550 2700
+	1    0    0    -1
+$EndComp
+Wire Wire Line
+	6350 2600 6350 2650
+Wire Wire Line
+	6250 2750 6250 3500
+Wire Wire Line
+	6250 2750 6350 2750
 $EndSCHEMATC
