File: GPIO.sch (KiCad schematic (older format))
At the start: 27 parts

Commit message: Add files via upload
Parts:
- D1, D2, D3, D4, D5, D6, D7, D8: renamed from D?; footprint (none) -> LEDs:LED-3MM
- P5, P6: renamed from P?; footprint (none) -> Pin_Headers:Pin_Header_Straight_1x08
- R2, R3, R4, R5, R6, R7, R8, R9: renamed from R?; footprint (none) -> Resistors_ThroughHole:Resistor_Horizontal_RM10mm
- RR2: renamed from RR?; footprint (none) -> Resistors_ThroughHole:Resistor_Array_SIP8
- SW2, SW3, SW4, SW5, SW6, SW7, SW8, SW9: renamed from SW?; footprint (none) -> Buttons_Switches_ThroughHole:Push_button_2_pin
Changed lines of the file:
@@
 EESchema Schematic File Version 2
+LIBS:8051_dev-rescue
 LIBS:power
 LIBS:device
@@
 LIBS:contrib
 LIBS:valves
-LIBS:8051_generic_89s51
 LIBS:7805_mod
-LIBS:HexConverter
-LIBS:MOTOR
-LIBS:ams1117_
-LIBS:arduinoNano
-LIBS:arduinouno
-LIBS:buzzer
-LIBS:cmos_cell
-LIBS:color_sensor
-LIBS:esp8266
-LIBS:fingerprintsensor
-LIBS:flex
-LIBS:ftdi232rl
-LIBS:hexconverter
-LIBS:i2cmemoty24ls256
-LIBS:l293d_modified
-LIBS:ldr
-LIBS:lm3915
-LIBS:oleddisplay
-LIBS:ov7670
-LIBS:pushbutton
-LIBS:relay
-LIBS:sd_card_module
-LIBS:servo
-LIBS:valve
-LIBS:xbee
-LIBS:max_232
-LIBS:0808
 LIBS:8051_dev-cache
 EELAYER 25 0
@@
 $Descr A4 11693 8268
 encoding utf-8
-Sheet 3 9
+Sheet 3 10
 Title ""
 Date ""
@@
 $EndDescr
 $Comp
-L LED D?
+L LED D1
 U 1 1 579AE4EE
 P 3650 2300
-F 0 "D?" H 3650 2400 50  0000 C CNN
+F 0 "D1" H 3650 2400 50  0000 C CNN
 F 1 "LED" H 3650 2200 50  0000 C CNN
-F 2 "" H 3650 2300 50  0000 C CNN
+F 2 "LEDs:LED-3MM" H 3650 2300 50  0001 C CNN
 F 3 "" H 3650 2300 50  0000 C CNN
 	1    3650 2300
@@
 $EndComp
 $Comp
-L R R?
+L R R2
 U 1 1 579AE6C3
 P 2850 2300
-F 0 "R?" V 2930 2300 50  0000 C CNN
+F 0 "R2" V 2930 2300 50  0000 C CNN
 F 1 "330" V 2850 2300 50  0000 C CNN
-F 2 "" V 2780 2300 50  0000 C CNN
+F 2 "Resistors_ThroughHole:Resistor_Horizontal_RM10mm" V 2780 2300 50  0001 C CNN
 F 3 "" H 2850 2300 50  0000 C CNN
 	1    2850 2300
@@
 $EndComp
 $Comp
-L LED D?
+L LED D2
 U 1 1 579AEAA2
 P 3650 2700
-F 0 "D?" H 3650 2800 50  0000 C CNN
+F 0 "D2" H 3650 2800 50  0000 C CNN
 F 1 "LED" H 3650 2600 50  0000 C CNN
-F 2 "" H 3650 2700 50  0000 C CNN
+F 2 "LEDs:LED-3MM" H 3650 2700 50  0001 C CNN
 F 3 "" H 3650 2700 50  0000 C CNN
 	1    3650 2700
@@
 $EndComp
 $Comp
-L R R?
+L R R3
 U 1 1 579AEAA8
 P 2850 2700
-F 0 "R?" V 2930 2700 50  0000 C CNN
+F 0 "R3" V 2930 2700 50  0000 C CNN
 F 1 "330" V 2850 2700 50  0000 C CNN
-F 2 "" V 2780 2700 50  0000 C CNN
+F 2 "Resistors_ThroughHole:Resistor_Horizontal_RM10mm" V 2780 2700 50  0001 C CNN
 F 3 "" H 2850 2700 50  0000 C CNN
 	1    2850 2700
@@
 $EndComp
 $Comp
-L LED D?
+L LED D3
 U 1 1 579AEB1B
 P 3650 3100
-F 0 "D?" H 3650 3200 50  0000 C CNN
+F 0 "D3" H 3650 3200 50  0000 C CNN
 F 1 "LED" H 3650 3000 50  0000 C CNN
-F 2 "" H 3650 3100 50  0000 C CNN
+F 2 "LEDs:LED-3MM" H 3650 3100 50  0001 C CNN
 F 3 "" H 3650 3100 50  0000 C CNN
 	1    3650 3100
@@
 $EndComp
 $Comp
-L R R?
+L R R4
 U 1 1 579AEB21
 P 2850 3100
-F 0 "R?" V 2930 3100 50  0000 C CNN
+F 0 "R4" V 2930 3100 50  0000 C CNN
 F 1 "330" V 2850 3100 50  0000 C CNN
-F 2 "" V 2780 3100 50  0000 C CNN
+F 2 "Resistors_ThroughHole:Resistor_Horizontal_RM10mm" V 2780 3100 50  0001 C CNN
 F 3 "" H 2850 3100 50  0000 C CNN
 	1    2850 3100
@@
 $EndComp
 $Comp
-L LED D?
+L LED D4
 U 1 1 579AEB28
 P 3650 3500
-F 0 "D?" H 3650 3600 50  0000 C CNN
+F 0 "D4" H 3650 3600 50  0000 C CNN
 F 1 "LED" H 3650 3400 50  0000 C CNN
-F 2 "" H 3650 3500 50  0000 C CNN
+F 2 "LEDs:LED-3MM" H 3650 3500 50  0001 C CNN
 F 3 "" H 3650 3500 50  0000 C CNN
 	1    3650 3500
@@
 $EndComp
 $Comp
-L R R?
+L R R5
 U 1 1 579AEB2E
 P 2850 3500
-F 0 "R?" V 2930 3500 50  0000 C CNN
+F 0 "R5" V 2930 3500 50  0000 C CNN
 F 1 "330" V 2850 3500 50  0000 C CNN
-F 2 "" V 2780 3500 50  0000 C CNN
+F 2 "Resistors_ThroughHole:Resistor_Horizontal_RM10mm" V 2780 3500 50  0001 C CNN
 F 3 "" H 2850 3500 50  0000 C CNN
 	1    2850 3500
@@
 $EndComp
 $Comp
-L LED D?
+L LED D5
 U 1 1 579AED35
 P 3650 3800
-F 0 "D?" H 3650 3900 50  0000 C CNN
+F 0 "D5" H 3650 3900 50  0000 C CNN
 F 1 "LED" H 3650 3700 50  0000 C CNN
-F 2 "" H 3650 3800 50  0000 C CNN
+F 2 "LEDs:LED-3MM" H 3650 3800 50  0001 C CNN
 F 3 "" H 3650 3800 50  0000 C CNN
 	1    3650 3800
@@
 $EndComp
 $Comp
-L R R?
+L R R6
 U 1 1 579AED3B
 P 2850 3800
-F 0 "R?" V 2930 3800 50  0000 C CNN
+F 0 "R6" V 2930 3800 50  0000 C CNN
 F 1 "330" V 2850 3800 50  0000 C CNN
-F 2 "" V 2780 3800 50  0000 C CNN
+F 2 "Resistors_ThroughHole:Resistor_Horizontal_RM10mm" V 2780 3800 50  0001 C CNN
 F 3 "" H 2850 3800 50  0000 C CNN
 	1    2850 3800
@@
 $EndComp
 $Comp
-L LED D?
+L LED D6
 U 1 1 579AED42
 P 3650 4200
-F 0 "D?" H 3650 4300 50  0000 C CNN
+F 0 "D6" H 3650 4300 50  0000 C CNN
 F 1 "LED" H 3650 4100 50  0000 C CNN
-F 2 "" H 3650 4200 50  0000 C CNN
+F 2 "LEDs:LED-3MM" H 3650 4200 50  0001 C CNN
 F 3 "" H 3650 4200 50  0000 C CNN
 	1    3650 4200
@@
 $EndComp
 $Comp
-L R R?
+L R R7
 U 1 1 579AED48
 P 2850 4200
-F 0 "R?" V 2930 4200 50  0000 C CNN
+F 0 "R7" V 2930 4200 50  0000 C CNN
 F 1 "330" V 2850 4200 50  0000 C CNN
-F 2 "" V 2780 4200 50  0000 C CNN
+F 2 "Resistors_ThroughHole:Resistor_Horizontal_RM10mm" V 2780 4200 50  0001 C CNN
 F 3 "" H 2850 4200 50  0000 C CNN
 	1    2850 4200
@@
 $EndComp
 $Comp
-L LED D?
+L LED D7
 U 1 1 579AED4F
 P 3650 4600
-F 0 "D?" H 3650 4700 50  0000 C CNN
+F 0 "D7" H 3650 4700 50  0000 C CNN
 F 1 "LED" H 3650 4500 50  0000 C CNN
-F 2 "" H 3650 4600 50  0000 C CNN
+F 2 "LEDs:LED-3MM" H 3650 4600 50  0001 C CNN
 F 3 "" H 3650 4600 50  0000 C CNN
 	1    3650 4600
@@
 $EndComp
 $Comp
-L R R?
+L R R8
 U 1 1 579AED55
 P 2850 4600
-F 0 "R?" V 2930 4600 50  0000 C CNN
+F 0 "R8" V 2930 4600 50  0000 C CNN
 F 1 "330" V 2850 4600 50  0000 C CNN
-F 2 "" V 2780 4600 50  0000 C CNN
+F 2 "Resistors_ThroughHole:Resistor_Horizontal_RM10mm" V 2780 4600 50  0001 C CNN
 F 3 "" H 2850 4600 50  0000 C CNN
 	1    2850 4600
@@
 $EndComp
 $Comp
-L LED D?
+L LED D8
 U 1 1 579AED5C
 P 3650 5000
-F 0 "D?" H 3650 5100 50  0000 C CNN
+F 0 "D8" H 3650 5100 50  0000 C CNN
 F 1 "LED" H 3650 4900 50  0000 C CNN
-F 2 "" H 3650 5000 50  0000 C CNN
+F 2 "LEDs:LED-3MM" H 3650 5000 50  0001 C CNN
 F 3 "" H 3650 5000 50  0000 C CNN
 	1    3650 5000
@@
 $EndComp
 $Comp
-L R R?
+L R R9
 U 1 1 579AED62
 P 2850 5000
-F 0 "R?" V 2930 5000 50  0000 C CNN
+F 0 "R9" V 2930 5000 50  0000 C CNN
 F 1 "330" V 2850 5000 50  0000 C CNN
-F 2 "" V 2780 5000 50  0000 C CNN
+F 2 "Resistors_ThroughHole:Resistor_Horizontal_RM10mm" V 2780 5000 50  0001 C CNN
 F 3 "" H 2850 5000 50  0000 C CNN
 	1    2850 5000
@@
 GPIO_GND
 $Comp
-L CONN_01X08 P?
+L CONN_01X08 P5
 U 1 1 579AEFA4
 P 1350 3650
-F 0 "P?" H 1350 4100 50  0000 C CNN
+F 0 "P5" H 1350 4100 50  0000 C CNN
 F 1 "GPIO_LED_HEADERS" V 1450 3650 50  0000 C CNN
-F 2 "" H 1350 3650 50  0000 C CNN
+F 2 "Pin_Headers:Pin_Header_Straight_1x08" H 1350 3650 50  0001 C CNN
 F 3 "" H 1350 3650 50  0000 C CNN
 	1    1350 3650
@@
 $EndComp
 $Comp
-L RR8 RR?
+L RR8 RR2
 U 1 1 579B08B6
 P 7200 3750
-F 0 "RR?" H 7250 4300 50  0000 C CNN
+F 0 "RR2" H 7250 4300 50  0000 C CNN
 F 1 "RR8" V 7230 3750 50  0000 C CNN
-F 2 "" H 7200 3750 50  0000 C CNN
+F 2 "Resistors_ThroughHole:Resistor_Array_SIP8" H 7200 3750 50  0001 C CNN
 F 3 "" H 7200 3750 50  0000 C CNN
 	1    7200 3750
@@
 GPIO_VCC
 $Comp
-L CONN_01X08 P?
+L CONN_01X08 P6
 U 1 1 579B1533
 P 6150 3750
-F 0 "P?" H 6150 4200 50  0000 C CNN
+F 0 "P6" H 6150 4200 50  0000 C CNN
 F 1 "GPIO_SWITCHES_HEADER" V 6250 3750 50  0000 C CNN
-F 2 "" H 6150 3750 50  0000 C CNN
+F 2 "Pin_Headers:Pin_Header_Straight_1x08" H 6150 3750 50  0001 C CNN
 F 3 "" H 6150 3750 50  0000 C CNN
 	1    6150 3750
@@
 $EndComp
 $Comp
-L SW_PUSH SW?
+L SW_PUSH SW2
 U 1 1 579B17C2
 P 8100 3100
-F 0 "SW?" H 8250 3210 50  0000 C CNN
+F 0 "SW2" H 8250 3210 50  0000 C CNN
 F 1 "SW_PUSH" H 8100 3020 50  0000 C CNN
-F 2 "" H 8100 3100 50  0000 C CNN
+F 2 "Buttons_Switches_ThroughHole:Push_button_2_pin" H 8100 3100 50  0001 C CNN
 F 3 "" H 8100 3100 50  0000 C CNN
 	1    8100 3100
@@
 $EndComp
 $Comp
-L SW_PUSH SW?
+L SW_PUSH SW3
 U 1 1 579B182F
 P 8100 3350
-F 0 "SW?" H 8250 3460 50  0000 C CNN
+F 0 "SW3" H 8250 3460 50  0000 C CNN
 F 1 "SW_PUSH" H 8100 3270 50  0000 C CNN
-F 2 "" H 8100 3350 50  0000 C CNN
+F 2 "Buttons_Switches_ThroughHole:Push_button_2_pin" H 8100 3350 50  0001 C CNN
 F 3 "" H 8100 3350 50  0000 C CNN
 	1    8100 3350
@@
 $EndComp
 $Comp
-L SW_PUSH SW?
+L SW_PUSH SW4
 U 1 1 579B1882
 P 8100 3600
-F 0 "SW?" H 8250 3710 50  0000 C CNN
+F 0 "SW4" H 8250 3710 50  0000 C CNN
 F 1 "SW_PUSH" H 8100 3520 50  0000 C CNN
-F 2 "" H 8100 3600 50  0000 C CNN
+F 2 "Buttons_Switches_ThroughHole:Push_button_2_pin" H 8100 3600 50  0001 C CNN
 F 3 "" H 8100 3600 50  0000 C CNN
 	1    8100 3600
@@
 $EndComp
 $Comp
-L SW_PUSH SW?
+L SW_PUSH SW5
 U 1 1 579B18D5
 P 8100 3800
-F 0 "SW?" H 8250 3910 50  0000 C CNN
+F 0 "SW5" H 8250 3910 50  0000 C CNN
 F 1 "SW_PUSH" H 8100 3720 50  0000 C CNN
-F 2 "" H 8100 3800 50  0000 C CNN
+F 2 "Buttons_Switches_ThroughHole:Push_button_2_pin" H 8100 3800 50  0001 C CNN
 F 3 "" H 8100 3800 50  0000 C CNN
 	1    8100 3800
@@
 $EndComp
 $Comp
-L SW_PUSH SW?
+L SW_PUSH SW6
 U 1 1 579B1920
 P 8100 4000
-F 0 "SW?" H 8250 4110 50  0000 C CNN
+F 0 "SW6" H 8250 4110 50  0000 C CNN
 F 1 "SW_PUSH" H 8100 3920 50  0000 C CNN
-F 2 "" H 8100 4000 50  0000 C CNN
+F 2 "Buttons_Switches_ThroughHole:Push_button_2_pin" H 8100 4000 50  0001 C CNN
 F 3 "" H 8100 4000 50  0000 C CNN
 	1    8100 4000
@@
 $EndComp
 $Comp
-L SW_PUSH SW?
+L SW_PUSH SW7
 U 1 1 579B1979
 P 8100 4200
-F 0 "SW?" H 8250 4310 50  0000 C CNN
+F 0 "SW7" H 8250 4310 50  0000 C CNN
 F 1 "SW_PUSH" H 8100 4120 50  0000 C CNN
-F 2 "" H 8100 4200 50  0000 C CNN
+F 2 "Buttons_Switches_ThroughHole:Push_button_2_pin" H 8100 4200 50  0001 C CNN
 F 3 "" H 8100 4200 50  0000 C CNN
 	1    8100 4200
@@
 $EndComp
 $Comp
-L SW_PUSH SW?
+L SW_PUSH SW8
 U 1 1 579B19C0
 P 8100 4400
-F 0 "SW?" H 8250 4510 50  0000 C CNN
+F 0 "SW8" H 8250 4510 50  0000 C CNN
 F 1 "SW_PUSH" H 8100 4320 50  0000 C CNN
-F 2 "" H 8100 4400 50  0000 C CNN
+F 2 "Buttons_Switches_ThroughHole:Push_button_2_pin" H 8100 4400 50  0001 C CNN
 F 3 "" H 8100 4400 50  0000 C CNN
 	1    8100 4400
@@
 $EndComp
 $Comp
-L SW_PUSH SW?
+L SW_PUSH SW9
 U 1 1 579B1A0B
 P 8100 4600
-F 0 "SW?" H 8250 4710 50  0000 C CNN
+F 0 "SW9" H 8250 4710 50  0000 C CNN
 F 1 "SW_PUSH" H 8100 4520 50  0000 C CNN
-F 2 "" H 8100 4600 50  0000 C CNN
+F 2 "Buttons_Switches_ThroughHole:Push_button_2_pin" H 8100 4600 50  0001 C CNN
 F 3 "" H 8100 4600 50  0000 C CNN
 	1    8100 4600
