File: LCD.sch (KiCad schematic (older format))
At the start: 4 parts

Commit message: Add files via upload
Parts:
- added P8: LCD_power_head, Pin_Headers:Pin_Header_Straight_1x02, symbol CONN_01X02
- DS1: renamed from DS?; footprint WC1602A -> Display:WC1602A
- P7: renamed from P?; footprint (none) -> Pin_Headers:Pin_Header_Straight_1x11
- R10: renamed from R?; footprint (none) -> Resistors_ThroughHole:Resistor_Horizontal_RM10mm
- RV1: renamed from RV?; footprint (none) -> Potentiometers:Potentiometer_Trimmer-Suntan-TSR-3386P
Connections:
- net LCD_GND: now also P8.1 (P1)
- net LCD_VCC: now also P8.2 (P2)
Changed lines of the file:
@@
 EESchema Schematic File Version 2
+LIBS:8051_dev-rescue
 LIBS:power
 LIBS:device
@@
 LIBS:contrib
 LIBS:valves
-LIBS:8051_generic_89s51
 LIBS:7805_mod
-LIBS:HexConverter
-LIBS:MOTOR
-LIBS:ams1117_
-LIBS:arduinoNano
-LIBS:arduinouno
-LIBS:buzzer
-LIBS:cmos_cell
-LIBS:color_sensor
-LIBS:esp8266
-LIBS:fingerprintsensor
-LIBS:flex
-LIBS:ftdi232rl
-LIBS:hexconverter
-LIBS:i2cmemoty24ls256
-LIBS:l293d_modified
-LIBS:ldr
-LIBS:lm3915
-LIBS:oleddisplay
-LIBS:ov7670
-LIBS:pushbutton
-LIBS:relay
-LIBS:sd_card_module
-LIBS:servo
-LIBS:valve
-LIBS:xbee
-LIBS:max_232
-LIBS:0808
 LIBS:8051_dev-cache
 EELAYER 25 0
@@
 $Descr A4 11693 8268
 encoding utf-8
-Sheet 4 9
+Sheet 3 10
 Title ""
 Date ""
@@
 $EndDescr
 $Comp
-L LCD16X2 DS?
+L LCD16X2 DS1
 U 1 1 579AF51D
 P 5500 2800
-F 0 "DS?" H 4700 3200 50  0000 C CNN
+F 0 "DS1" H 4700 3200 50  0000 C CNN
 F 1 "LCD16X2" H 6200 3200 50  0000 C CNN
-F 2 "WC1602A" H 5500 2750 50  0000 C CIN
+F 2 "Display:WC1602A" H 5500 2750 50  0000 C CIN
 F 3 "" H 5500 2800 50  0000 C CNN
 	1    5500 2800
 	1    0    0    -1
 $EndComp
-Text HLabel 4000 3450 0    60   Input Italic 0
+Text GLabel 4300 3300 0    60   Input Italic 0
+LCD_VCC
+Text GLabel 3900 4350 0    60   Input Italic 0
 LCD_GND
-Text HLabel 4500 3600 0    60   Input Italic 0
-LCD_VCC
-Wire Wire Line
-	4000 3450 4750 3450
+$Comp
+L R R10
+U 1 1 579AF6A8
+P 6150 3550
+F 0 "R10" V 6230 3550 50  0000 C CNN
+F 1 "330" V 6150 3550 50  0000 C CNN
+F 2 "Resistors_ThroughHole:Resistor_Horizontal_RM10mm" V 6080 3550 50  0001 C CNN
+F 3 "" H 6150 3550 50  0000 C CNN
+	1    6150 3550
+	1    0    0    -1
+$EndComp
+$Comp
+L CONN_01X11 P7
+U 1 1 579AF733
+P 5550 4400
+F 0 "P7" H 5550 5000 50  0000 C CNN
+F 1 "LCD_PIN_HEADERS" V 5650 4400 50  0000 C CNN
+F 2 "Pin_Headers:Pin_Header_Straight_1x11" H 5550 4400 50  0001 C CNN
+F 3 "" H 5550 4400 50  0000 C CNN
+	1    5550 4400
+	0    1    1    0
+$EndComp
+$Comp
+L POT RV1
+U 1 1 579AF584
+P 4550 3900
+F 0 "RV1" H 4550 3820 50  0000 C CNN
+F 1 "POT" H 4550 3900 50  0000 C CNN
+F 2 "Potentiometers:Potentiometer_Trimmer-Suntan-TSR-3386P" H 4550 3900 50  0001 C CNN
+F 3 "" H 4550 3900 50  0000 C CNN
+	1    4550 3900
+	0    1    1    0
+$EndComp
+$Comp
+L CONN_01X02 P8
+U 1 1 57A5BEBF
+P 7800 4050
+F 0 "P8" H 7800 4200 50  0000 C CNN
+F 1 "LCD_power_head" V 7900 4050 50  0000 C CNN
+F 2 "Pin_Headers:Pin_Header_Straight_1x02" H 7800 4050 50  0001 C CNN
+F 3 "" H 7800 4050 50  0000 C CNN
+	1    7800 4050
+	1    0    0    -1
+$EndComp
 Wire Wire Line
 	4750 3450 4750 3300
@@
 	4300 3500 4300 3450
 Connection ~ 4300 3450
-Text GLabel 4300 3300 0    60   Input Italic 0
-LCD_VCC
 Wire Wire Line
 	4300 3300 4700 3300
-Text GLabel 3900 4350 0    60   Input Italic 0
-LCD_GND
 Wire Wire Line
 	3900 4350 4100 4350
@@
 	4100 4350 4100 4100
 Connection ~ 4100 4100
-Text GLabel 6500 3700 2    60   Input Italic 0
-LCD_VCC
-Text GLabel 6500 3500 2    60   Input Italic 0
-LCD_GND
-$Comp
-L R R?
-U 1 1 579AF6A8
-P 6150 3550
-F 0 "R?" V 6230 3550 50  0000 C CNN
-F 1 "330" V 6150 3550 50  0000 C CNN
-F 2 "" V 6080 3550 50  0000 C CNN
-F 3 "" H 6150 3550 50  0000 C CNN
-	1    6150 3550
-	1    0    0    -1
-$EndComp
 Wire Wire Line
 	6150 3400 6150 3300
 Wire Wire Line
-	6500 3500 6250 3500
+	6250 3500 7600 3500
 Wire Wire Line
 	6250 3500 6250 3300
 Wire Wire Line
-	6150 3700 6500 3700
-$Comp
-L CONN_01X11 P?
-U 1 1 579AF733
-P 5550 4400
-F 0 "P?" H 5550 5000 50  0000 C CNN
-F 1 "LCD_PIN_HEADERS" V 5650 4400 50  0000 C CNN
-F 2 "" H 5550 4400 50  0000 C CNN
-F 3 "" H 5550 4400 50  0000 C CNN
-	1    5550 4400
-	0    1    1    0
-$EndComp
-$Comp
-L POT RV?
-U 1 1 579AF584
-P 4550 3900
-F 0 "RV?" H 4550 3820 50  0000 C CNN
-F 1 "POT" H 4550 3900 50  0000 C CNN
-F 2 "" H 4550 3900 50  0000 C CNN
-F 3 "" H 4550 3900 50  0000 C CNN
-	1    4550 3900
-	0    1    1    0
-$EndComp
+	6150 3700 7350 3700
 Wire Wire Line
 	4950 3900 4700 3900
@@
 Wire Wire Line
 	6050 4200 6050 3300
+Wire Wire Line
+	7600 3500 7600 4000
+Wire Wire Line
+	7350 3700 7350 4100
+Wire Wire Line
+	7350 4100 7600 4100
+Wire Wire Line
+	4300 3450 4750 3450
+Text GLabel 7150 3900 0    60   Input ~ 0
+LCD_VCC
+Wire Wire Line
+	7150 3900 7350 3900
+Connection ~ 7350 3900
+Text GLabel 7050 3300 0    60   Input ~ 0
+LCD_GND
+Wire Wire Line
+	7050 3300 7350 3300
+Wire Wire Line
+	7350 3300 7350 3500
+Connection ~ 7350 3500
 $EndSCHEMATC
