File: POWER_SUPPLY.sch (KiCad schematic (older format))
At the start: 5 parts

Commit message: Add files via upload
Parts:
- removed U?: 7805_mod, symbol 7805_mod
- added P23: 9Vout, Pin_Headers:Pin_Header_Straight_1x02, symbol CONN_01X02
- added P24: 5V_Pin, Pin_Headers:Pin_Header_Straight_1x05, symbol CONN_01X05
- added P25: GND_pin, Pin_Headers:Pin_Header_Straight_1x05, symbol CONN_01X05
- added U5: 7805_mod, Connect:PINHEAD1-3, symbol 7805_mod
- C4, C5, C6: renamed from C?; footprint (none) -> Capacitors_ThroughHole:C_Disc_D3_P2.5
- CON1: renamed from CON?; footprint (none) -> Connect:BARREL_JACK
Connections:
- net labels added: 5V_pin, GND_pin
- wire segments 13 -> 30
Changed lines of the file:
@@
 EESchema Schematic File Version 2
+LIBS:8051_dev-rescue
 LIBS:power
 LIBS:device
@@
 LIBS:contrib
 LIBS:valves
-LIBS:8051_generic_89s51
 LIBS:7805_mod
-LIBS:HexConverter
-LIBS:MOTOR
-LIBS:ams1117_
-LIBS:arduinoNano
-LIBS:arduinouno
-LIBS:buzzer
-LIBS:cmos_cell
-LIBS:color_sensor
-LIBS:esp8266
-LIBS:fingerprintsensor
-LIBS:flex
-LIBS:ftdi232rl
-LIBS:hexconverter
-LIBS:i2cmemoty24ls256
-LIBS:l293d_modified
-LIBS:ldr
-LIBS:lm3915
-LIBS:oleddisplay
-LIBS:ov7670
-LIBS:pushbutton
-LIBS:relay
-LIBS:sd_card_module
-LIBS:servo
-LIBS:valve
-LIBS:xbee
-LIBS:max_232
-LIBS:0808
 LIBS:8051_dev-cache
 EELAYER 25 0
@@
 $Descr A4 11693 8268
 encoding utf-8
-Sheet 2 9
+Sheet 8 10
 Title ""
 Date ""
@@
 $EndDescr
 $Comp
-L BARREL_JACK CON?
+L BARREL_JACK CON1
 U 1 1 579ADE43
 P 3000 3450
-F 0 "CON?" H 3000 3700 50  0000 C CNN
+F 0 "CON1" H 3000 3700 50  0000 C CNN
 F 1 "BARREL_JACK" H 3000 3250 50  0000 C CNN
-F 2 "" H 3000 3450 50  0000 C CNN
+F 2 "Connect:BARREL_JACK" H 3000 3450 50  0001 C CNN
 F 3 "" H 3000 3450 50  0000 C CNN
 	1    3000 3450
@@
 $EndComp
 $Comp
-L 7805_mod U?
-U 1 1 579ADEDE
-P 4700 3550
-F 0 "U?" H 4700 3550 60  0000 C CNN
-F 1 "7805_mod" H 4850 4100 60  0000 C CNN
-F 2 "" H 4700 3550 60  0000 C CNN
-F 3 "" H 4700 3550 60  0000 C CNN
-	1    4700 3550
-	1    0    0    -1
-$EndComp
-$Comp
-L CP C?
+L CP C6
 U 1 1 579ADF07
 P 5300 3550
-F 0 "C?" H 5325 3650 50  0000 L CNN
+F 0 "C6" H 5325 3650 50  0000 L CNN
 F 1 "10Uf_63V" H 5325 3450 50  0000 L CNN
-F 2 "" H 5338 3400 50  0000 C CNN
+F 2 "Capacitors_ThroughHole:C_Disc_D3_P2.5" H 5338 3400 50  0001 C CNN
 F 3 "" H 5300 3550 50  0000 C CNN
 	1    5300 3550
@@
 $EndComp
 $Comp
-L CP C?
+L CP C5
 U 1 1 579ADF43
 P 4150 3600
-F 0 "C?" H 4175 3700 50  0000 L CNN
+F 0 "C5" H 4175 3700 50  0000 L CNN
 F 1 "1000UF_25V" H 4175 3500 50  0000 L CNN
-F 2 "" H 4188 3450 50  0000 C CNN
+F 2 "Capacitors_ThroughHole:C_Disc_D3_P2.5" H 4188 3450 50  0001 C CNN
 F 3 "" H 4150 3600 50  0000 C CNN
 	1    4150 3600
@@
 $EndComp
 $Comp
-L C C?
+L C C4
 U 1 1 579ADF77
 P 3700 3600
-F 0 "C?" H 3725 3700 50  0000 L CNN
+F 0 "C4" H 3725 3700 50  0000 L CNN
 F 1 "0.1UF" H 3725 3500 50  0000 L CNN
-F 2 "" H 3738 3450 50  0000 C CNN
+F 2 "Capacitors_ThroughHole:C_Disc_D3_P2.5" H 3738 3450 50  0001 C CNN
 F 3 "" H 3700 3600 50  0000 C CNN
 	1    3700 3600
@@
 	5850 3250 5300 3250
 Connection ~ 5300 3250
+$Comp
+L 7805_mod U5
+U 1 1 57A61DF1
+P 4700 3550
+F 0 "U5" H 4700 3550 60  0000 C CNN
+F 1 "7805_mod" H 4700 3550 60  0000 C CNN
+F 2 "Connect:PINHEAD1-3" H 4700 3550 60  0001 C CNN
+F 3 "" H 4700 3550 60  0000 C CNN
+	1    4700 3550
+	1    0    0    -1
+$EndComp
+Wire Wire Line
+	5850 3850 5300 3850
+Connection ~ 5300 3850
+$Comp
+L CONN_01X02 P23
+U 1 1 57A5C281
+P 4200 2500
+F 0 "P23" H 4200 2650 50  0000 C CNN
+F 1 "9Vout" V 4300 2500 50  0000 C CNN
+F 2 "Pin_Headers:Pin_Header_Straight_1x02" H 4200 2500 50  0001 C CNN
+F 3 "" H 4200 2500 50  0000 C CNN
+	1    4200 2500
+	1    0    0    -1
+$EndComp
+Wire Wire Line
+	4000 2450 3500 2450
+Wire Wire Line
+	3500 2450 3500 3200
+Connection ~ 3500 3200
+Wire Wire Line
+	4000 2550 4000 3900
+Connection ~ 4000 3900
+$Comp
+L CONN_01X05 P24
+U 1 1 57A5C672
+P 5950 2050
+F 0 "P24" H 5950 2350 50  0000 C CNN
+F 1 "5V_Pin" V 6050 2050 50  0000 C CNN
+F 2 "Pin_Headers:Pin_Header_Straight_1x05" H 5950 2050 50  0001 C CNN
+F 3 "" H 5950 2050 50  0000 C CNN
+	1    5950 2050
+	0    -1   -1   0
+$EndComp
+Text GLabel 5150 2300 0    60   Input ~ 0
+5V_pin
+Text GLabel 5900 3400 2    60   Input ~ 0
+5V_pin
+Wire Wire Line
+	5900 3400 5600 3400
+Wire Wire Line
+	5600 3400 5600 3250
+Connection ~ 5600 3250
+Text GLabel 5200 2500 0    60   Input ~ 0
+GND_pin
+Wire Wire Line
+	5150 2300 6150 2300
+Wire Wire Line
+	6150 2300 6150 2250
+Wire Wire Line
+	6050 2250 6050 2300
+Connection ~ 6050 2300
+Wire Wire Line
+	5950 2250 5950 2300
+Connection ~ 5950 2300
+Wire Wire Line
+	5850 2250 5850 2300
+Connection ~ 5850 2300
+Wire Wire Line
+	5750 2250 5750 2300
+Connection ~ 5750 2300
+$Comp
+L CONN_01X05 P25
+U 1 1 57A5C82C
+P 5950 2700
+F 0 "P25" H 5950 3000 50  0000 C CNN
+F 1 "GND_pin" V 6050 2700 50  0000 C CNN
+F 2 "Pin_Headers:Pin_Header_Straight_1x05" H 5950 2700 50  0001 C CNN
+F 3 "" H 5950 2700 50  0000 C CNN
+	1    5950 2700
+	0    1    1    0
+$EndComp
+Wire Wire Line
+	6150 2500 5200 2500
+Connection ~ 5750 2500
+Connection ~ 5850 2500
+Connection ~ 5950 2500
+Connection ~ 6050 2500
+Connection ~ 6150 2500
+Connection ~ 6150 2300
+Text GLabel 5450 4100 0    60   Input ~ 0
+GND_pin
+Wire Wire Line
+	5450 4100 5600 4100
+Wire Wire Line
+	5600 4100 5600 3900
+Wire Wire Line
+	5600 3900 5550 3900
+Wire Wire Line
+	5550 3900 5550 3850
+Connection ~ 5550 3850
 $EndSCHEMATC
